File: pcb/spaceapi-map.kicad_sch (KiCad schematic)
At the start: 0 parts

Commit message: adding all symbols to schematic
Parts:
- added D1, D10, D11, D12, D13, D14, D15, D16, D17, D18, D19, D2, D20, D21, D22, D23, D24, D25, D26, D27, D28, D29, D3, D30, D31, D32, D33, D34, D35, D36, D37, D38, D39, D4, D40, D41, D42, D43, D44, D45, D46, D47, D48, D49, D5, D50, D51, D52, D53, D54, D55, D56, D57, D58, D59, D6, D60, D61, D62, D63, D64, D65, D66, D67, D68, D69, D7, D70, D71, D72, D73, D74, D75, D76, D77, D78, D79, D8, D80, D81, D82, D83, D9: WS2812B-2020, LED_SMD:LED_WS2812B-2020_PLCC4_2.0x2.0mm, symbol LED:WS2812B-2020
- added R1: 200, symbol Device:R
- added R2: LDR07, OptoDevice:R_LDR_5.1x4.3mm_P3.4mm_Vertical, symbol Sensor_Optical:LDR07
- added R3, R4: 47k, symbol Device:R
- added U1: ~, esp-devboard:ESP32C3, symbol esp-devboard:ESP32C3
Connections:
- new net: D4.1 (DOUT), D5.3 (DIN)
- new net: D3.1 (DOUT), D4.3 (DIN)
- new net: D73.1 (DOUT), D74.3 (DIN)
- new net: D72.1 (DOUT), D73.3 (DIN)
- new net: R1.1, U1.9 (D0)
- new net: D32.1 (DOUT), D33.3 (DIN)
- new net: D31.1 (DOUT), D32.3 (DIN)
- new net: D70.1 (DOUT), D71.3 (DIN)
- new net: D69.1 (DOUT), D70.3 (DIN)
- new net: D57.1 (DOUT), D58.3 (DIN)
- new net: D56.1 (DOUT), D57.3 (DIN)
- new net: D42.1 (DOUT), D43.3 (DIN)
- new net: D41.1 (DOUT), D42.3 (DIN)
- new net: D16.1 (DOUT), D17.3 (DIN)
- new net: D15.1 (DOUT), D16.3 (DIN)
- new net: D71.1 (DOUT), D72.3 (DIN)
- new net: D44.1 (DOUT), D45.3 (DIN)
- new net: D43.1 (DOUT), D44.3 (DIN)
- new net: D63.1 (DOUT), D64.3 (DIN)
- new net: D62.1 (DOUT), D63.3 (DIN)
- new net: D40.1 (DOUT), D41.3 (DIN)
- new net: D35.1 (DOUT), D36.3 (DIN)
- new net: D34.1 (DOUT), D35.3 (DIN)
- new net: D5.1 (DOUT), D6.3 (DIN)
- new net: D2.1 (DOUT), D3.3 (DIN)
- new net: D1.1 (DOUT), D2.3 (DIN)
- new net: D21.1 (DOUT), D22.3 (DIN)
- new net: D20.1 (DOUT), D21.3 (DIN)
- new net: D10.3 (DIN), D9.1 (DOUT)
- new net: D8.1 (DOUT), D9.3 (DIN)
- new net: D67.1 (DOUT), D68.3 (DIN)
- new net: D66.1 (DOUT), D67.3 (DIN)
- new net: D19.1 (DOUT), D20.3 (DIN)
- new net: D18.1 (DOUT), D19.3 (DIN)
- new net: D17.1 (DOUT), D18.3 (DIN)
- new net: D58.1 (DOUT), D59.3 (DIN)
- new net: D50.1 (DOUT), D51.3 (DIN)
- new net: D49.1 (DOUT), D50.3 (DIN)
- new net: D52.1 (DOUT), D53.3 (DIN)
- new net: D51.1 (DOUT), D52.3 (DIN)
- new net: D68.1 (DOUT), D69.3 (DIN)
- new net: D14.1 (DOUT), D15.3 (DIN)
- new net: D13.1 (DOUT), D14.3 (DIN)
- new net: D26.1 (DOUT), D27.3 (DIN)
- new net: D25.1 (DOUT), D26.3 (DIN)
- new net: D55.1 (DOUT), D56.3 (DIN)
- new net: D29.1 (DOUT), D30.3 (DIN)
- new net: D28.1 (DOUT), D29.3 (DIN)
- new net: D54.1 (DOUT), D55.3 (DIN)
- new net: D53.1 (DOUT), D54.3 (DIN)
- new net: D78.1 (DOUT), D79.3 (DIN)
- new net: D77.1 (DOUT), D78.3 (DIN)
- new net: D39.1 (DOUT), D40.3 (DIN)
- new net: D37.1 (DOUT), D38.3 (DIN)
- new net: D36.1 (DOUT), D37.3 (DIN)
- new net: D27.1 (DOUT), D28.3 (DIN)
- new net: D74.1 (DOUT), D75.3 (DIN)
- new net: D59.1 (DOUT), D60.3 (DIN)
- new net: D65.1 (DOUT), D66.3 (DIN)
- new net: D81.1 (DOUT), D82.3 (DIN)
- new net: D80.1 (DOUT), D81.3 (DIN)
- new net: D64.1 (DOUT), D65.3 (DIN)
- new net: D61.1 (DOUT), D62.3 (DIN)
- new net: D12.1 (DOUT), D13.3 (DIN)
- new net: D7.1 (DOUT), D8.3 (DIN)
- new net: D6.1 (DOUT), D7.3 (DIN)
- new net: D33.1 (DOUT), D34.3 (DIN)
- new net: D75.1 (DOUT), D76.3 (DIN)
- new net: D30.1 (DOUT), D31.3 (DIN)
- new net: D24.1 (DOUT), D25.3 (DIN)
- new net: D23.1 (DOUT), D24.3 (DIN)
- new net: D11.1 (DOUT), D12.3 (DIN)
- new net: D10.1 (DOUT), D11.3 (DIN)
- new net: D76.1 (DOUT), D77.3 (DIN)
- new net: D38.1 (DOUT), D39.3 (DIN)
- new net: D79.1 (DOUT), D80.3 (DIN)
- new net: D60.1 (DOUT), D61.3 (DIN)
- new net: D48.1 (DOUT), D49.3 (DIN)
- new net: D46.1 (DOUT), D47.3 (DIN)
- new net: D45.1 (DOUT), D46.3 (DIN)
- new net: D22.1 (DOUT), D23.3 (DIN)
- new net: D82.1 (DOUT), D83.3 (DIN)
- new net: D47.1 (DOUT), D48.3 (DIN)
- new net +5V: D1.4 (VDD), D10.4 (VDD), D11.4 (VDD), D12.4 (VDD), D13.4 (VDD), D14.4 (VDD), D15.4 (VDD), D16.4 (VDD), D17.4 (VDD), D18.4 (VDD), D19.4 (VDD), D2.4 (VDD), D20.4 (VDD), D21.4 (VDD), D22.4 (VDD), D23.4 (VDD), D24.4 (VDD), D25.4 (VDD), D26.4 (VDD), D27.4 (VDD), D28.4 (VDD), D29.4 (VDD), D3.4 (VDD), D30.4 (VDD), D31.4 (VDD), D32.4 (VDD), D33.4 (VDD), D34.4 (VDD), D35.4 (VDD), D36.4 (VDD), D37.4 (VDD), D38.4 (VDD), D39.4 (VDD), D4.4 (VDD), D40.4 (VDD), D41.4 (VDD), D42.4 (VDD), D43.4 (VDD), D44.4 (VDD), D45.4 (VDD), D46.4 (VDD), D47.4 (VDD), D48.4 (VDD), D49.4 (VDD), D5.4 (VDD), D50.4 (VDD), D51.4 (VDD), D52.4 (VDD), D53.4 (VDD), D54.4 (VDD), D55.4 (VDD), D56.4 (VDD), D57.4 (VDD), D58.4 (VDD), D59.4 (VDD), D6.4 (VDD), D60.4 (VDD), D61.4 (VDD), D62.4 (VDD), D63.4 (VDD), D64.4 (VDD), D65.4 (VDD), D66.4 (VDD), D67.4 (VDD), D68.4 (VDD), D69.4 (VDD), D7.4 (VDD), D70.4 (VDD), D71.4 (VDD), D72.4 (VDD), D73.4 (VDD), D74.4 (VDD), D75.4 (VDD), D76.4 (VDD), D77.4 (VDD), D78.4 (VDD), D79.4 (VDD), D8.4 (VDD), D80.4 (VDD), D81.4 (VDD), D82.4 (VDD), D83.4 (VDD), D9.4 (VDD), R4.1, U1.16 (5V)
- new net Din: D1.3 (DIN), R1.2
- new net GND: D1.2 (VSS), D10.2 (VSS), D11.2 (VSS), D12.2 (VSS), D13.2 (VSS), D14.2 (VSS), D15.2 (VSS), D16.2 (VSS), D17.2 (VSS), D18.2 (VSS), D19.2 (VSS), D2.2 (VSS), D20.2 (VSS), D21.2 (VSS), D22.2 (VSS), D23.2 (VSS), D24.2 (VSS), D25.2 (VSS), D26.2 (VSS), D27.2 (VSS), D28.2 (VSS), D29.2 (VSS), D3.2 (VSS), D30.2 (VSS), D31.2 (VSS), D32.2 (VSS), D33.2 (VSS), D34.2 (VSS), D35.2 (VSS), D36.2 (VSS), D37.2 (VSS), D38.2 (VSS), D39.2 (VSS), D4.2 (VSS), D40.2 (VSS), D41.2 (VSS), D42.2 (VSS), D43.2 (VSS), D44.2 (VSS), D45.2 (VSS), D46.2 (VSS), D47.2 (VSS), D48.2 (VSS), D49.2 (VSS), D5.2 (VSS), D50.2 (VSS), D51.2 (VSS), D52.2 (VSS), D53.2 (VSS), D54.2 (VSS), D55.2 (VSS), D56.2 (VSS), D57.2 (VSS), D58.2 (VSS), D59.2 (VSS), D6.2 (VSS), D60.2 (VSS), D61.2 (VSS), D62.2 (VSS), D63.2 (VSS), D64.2 (VSS), D65.2 (VSS), D66.2 (VSS), D67.2 (VSS), D68.2 (VSS), D69.2 (VSS), D7.2 (VSS), D70.2 (VSS), D71.2 (VSS), D72.2 (VSS), D73.2 (VSS), D74.2 (VSS), D75.2 (VSS), D76.2 (VSS), D77.2 (VSS), D78.2 (VSS), D79.2 (VSS), D8.2 (VSS), D80.2 (VSS), D81.2 (VSS), D82.2 (VSS), D83.2 (VSS), D9.2 (VSS), R2.2, R3.2, U1.15 (GND)
- new net LDR: R2.1, R3.1, R4.2, U1.12 (D3)

Commit message: changing ws2812b footprint
Parts:
- D1, D10, D11, D12, D13, D14, D15, D16, D17, D18, D19, D2, D20, D21, D22, D23, D24, D25, D26, D27, D28, D29, D3, D30, D31, D32, D33, D34, D35, D36, D37, D38, D39, D4, D40, D41, D42, D43, D44, D45, D46, D47, D48, D49, D5, D50, D51, D52, D53, D54, D55, D56, D57, D58, D59, D6, D60, D61, D62, D63, D64, D65, D66, D67, D68, D69, D7, D70, D71, D72, D73, D74, D75, D76, D77, D78, D79, D8, D80, D81, D82, D83, D9: footprint LED_SMD:LED_WS2812B-2020_PLCC4_2.0x2.0mm -> esp-devboard:LED_WS2812B-2020_PLCC4_2.0x2.0mm

Commit message: routing led data lines
Parts:
- R1, R3, R4: footprint (none) -> Resistor_SMD:R_0603_1608Metric
Changed lines of the file:
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@@
 			)
 		)
-		(property "Footprint" ""
+		(property "Footprint" "Resistor_SMD:R_0603_1608Metric"
 			(at 62.23 64.008 90)
 			(effects
@@
 			)
 		)
-		(property "Footprint" ""
+		(property "Footprint" "Resistor_SMD:R_0603_1608Metric"
 			(at 54.102 132.08 90)
 			(effects
@@
 			)
 		)
-		(property "Footprint" ""
+		(property "Footprint" "Resistor_SMD:R_0603_1608Metric"
 			(at 54.102 147.32 90)
 			(effects
